File: hardware/pcb/frsky_dsmx_caddy.sch (KiCad schematic (older format))
At the start: 26 parts, among them P1 G9X, P2 Fr-Sky, P3 DSMX, Q1 BC847C, Q2 Si2319DS, Q3 Si2319DS, Q4 BC847C, U1 7805, U2 LN-6206-30

Commit message: Reference doc for SOT-223 500mA 78M05 regulator used on TX caddy.
Parts:
- removed D2: DIODESCH, symbol DIODESCH
- P1: symbol CONN_7 -> CONN_8
Connections:
- net +3.3V: no longer R1.1
- net Rx: now also P1.8 (P8); no longer P1.7 (P7)
- net Rxd: now also P1.7 (P7); no longer P1.6 (P6)
- new net DSM: P1.6 (P6), R1.1
Other:
- moved on the sheet: R1
Changed lines of the file:
@@
-EESchema Schematic File Version 2  date Sat 27 Oct 2012 12:35:31 AM NZDT
+EESchema Schematic File Version 2  date Tue 30 Oct 2012 08:21:28 PM NZDT
 LIBS:gruvin
 LIBS:power
@@
 Sheet 1 1
 Title "Fr-Sky / DSMX TX Moudle Caddy"
-Date "26 oct 2012"
+Date "30 oct 2012"
 Rev "2.0"
 Comp ""
@@
 Comment4 "Licensed under the TAPR Open Hardware License (see file,  LICENSE)"
 $EndDescr
-Connection ~ 9850 3000
-Wire Wire Line
-	9800 3000 9850 3000
+Text Label 1350 3200 0    60   ~ 0
+DSM
+Wire Wire Line
+	1250 3200 1750 3200
+Wire Wire Line
+	1750 3200 1750 4400
+Wire Wire Line
+	5250 1750 5250 2850
+Wire Wire Line
+	5250 2850 5250 3200
+Connection ~ 5250 2850
+Wire Wire Line
+	5350 2850 5250 2850
+Connection ~ 5250 1750
+Wire Wire Line
+	4750 2650 4750 2850
+Wire Wire Line
+	4750 3250 4750 3300
+Wire Wire Line
+	3800 3050 3800 3300
+Connection ~ 2550 2750
+Wire Wire Line
+	2550 2750 2550 3050
+Wire Wire Line
+	2550 3050 2700 3050
+Wire Wire Line
+	3100 2750 2550 2750
+Wire Wire Line
+	2550 2750 2350 2750
+Wire Wire Line
+	2350 3250 2350 3600
+Wire Wire Line
+	2350 3600 1250 3600
+Wire Wire Line
+	3500 4400 9850 4400
+Wire Wire Line
+	9850 4400 9850 3000
+Wire Wire Line
+	9850 3000 9850 2650
+Wire Wire Line
+	9850 2650 10150 2650
+Wire Wire Line
+	3800 3050 3900 3050
+Wire Wire Line
+	3800 3300 1250 3300
+Wire Wire Line
+	5450 2150 5450 2250
+Wire Wire Line
+	5450 2250 5450 2350
+Connection ~ 5450 2250
+Wire Wire Line
+	6150 4000 6150 3900
+Wire Wire Line
+	9000 4000 9000 3900
+Wire Wire Line
+	4450 4000 4450 4100
+Connection ~ 8600 3900
+Connection ~ 8600 3500
+Connection ~ 9000 3500
+Wire Wire Line
+	9000 3900 8600 3900
+Wire Wire Line
+	8600 3900 8000 3900
+Wire Wire Line
+	8000 3900 7400 3900
+Wire Wire Line
+	7400 3900 6750 3900
+Wire Wire Line
+	6750 3900 6150 3900
+Wire Wire Line
+	2150 2300 2150 3400
+Wire Wire Line
+	10150 2150 8950 2150
+Wire Wire Line
+	8950 2150 8950 2350
+Wire Wire Line
+	6250 1450 1750 1450
+Wire Wire Line
+	1750 1450 1750 3000
+Wire Wire Line
+	1750 3000 1250 3000
+Wire Wire Line
+	1250 3500 2800 3500
+Connection ~ 4450 3500
+Wire Wire Line
+	7600 3500 7400 3500
+Wire Wire Line
+	7400 3500 7150 3500
+Wire Wire Line
+	4450 3500 4450 3600
+Wire Wire Line
+	8400 3500 8600 3500
+Wire Wire Line
+	8600 3500 9000 3500
+Wire Wire Line
+	9000 3500 9250 3500
+Wire Wire Line
+	4550 1750 4000 1750
+Wire Wire Line
+	4000 1750 3600 1750
+Wire Wire Line
+	4750 2050 4750 2100
+Wire Wire Line
+	4750 2100 4750 2150
+Connection ~ 6750 3900
+Connection ~ 6150 3500
+Connection ~ 7400 3900
+Wire Wire Line
+	6250 1750 5450 1750
+Wire Wire Line
+	5450 1750 5250 1750
+Wire Wire Line
+	5250 1750 4950 1750
+Wire Wire Line
+	8000 3900 8000 3800
+Connection ~ 7400 3500
+Wire Wire Line
+	3600 1750 3600 3500
+Connection ~ 3600 3500
+Wire Wire Line
+	4600 2100 4750 2100
+Connection ~ 4750 2100
+Wire Wire Line
+	6250 1650 2150 1650
+Wire Wire Line
+	2150 3400 1250 3400
+Wire Wire Line
+	6250 1550 1900 1550
+Wire Wire Line
+	1900 1550 1900 3100
+Wire Wire Line
+	1900 3100 1250 3100
+Wire Wire Line
+	9250 3500 9250 3000
+Wire Wire Line
+	9250 3000 9250 2250
+Wire Wire Line
+	9250 2250 10150 2250
+Connection ~ 8000 3900
+Wire Wire Line
+	2150 1650 2150 1900
+Wire Wire Line
+	6350 3500 6150 3500
+Wire Wire Line
+	6150 3500 5450 3500
+Wire Wire Line
+	1250 3700 1400 3700
+Wire Wire Line
+	1400 3700 1400 3950
+Wire Wire Line
+	5450 2250 5900 2250
+Connection ~ 5450 1750
+Wire Wire Line
+	6750 3800 6750 3900
+Wire Wire Line
+	4100 2100 4000 2100
+Wire Wire Line
+	4000 2100 4000 1750
+Connection ~ 4000 1750
+Wire Wire Line
+	6250 1950 5900 1950
+Wire Wire Line
+	3400 2950 3400 3050
+Wire Wire Line
+	3400 3050 3400 3150
+Wire Wire Line
+	3400 2550 3400 2450
+Wire Wire Line
+	3400 1950 3400 1350
+Wire Wire Line
+	3400 1350 5750 1350
+Wire Wire Line
+	5750 1350 5750 1850
+Wire Wire Line
+	5750 1850 6250 1850
+Wire Wire Line
+	3200 3050 3400 3050
+Connection ~ 3400 3050
+Wire Wire Line
+	3300 3500 3600 3500
+Wire Wire Line
+	3600 3500 4450 3500
+Wire Wire Line
+	4450 3500 5050 3500
+Wire Wire Line
+	4450 3050 4400 3050
+Wire Wire Line
+	1750 4400 3000 4400
+Wire Wire Line
+	5850 2850 5900 2850
+Wire Wire Line
+	5900 2850 5900 2250
+Wire Wire Line
+	5900 2250 5900 1950
 Connection ~ 5900 2250
-Wire Wire Line
-	5900 2850 5900 1950
-Wire Wire Line
-	5900 2850 5850 2850
-Wire Wire Line
-	1750 3400 1750 4400
-Wire Wire Line
-	1750 4400 3100 4400
-Wire Wire Line
-	4450 3050 4400 3050
-Wire Wire Line
-	5050 3500 3300 3500
-Connection ~ 3400 3050
-Wire Wire Line
-	3200 3050 3400 3050
-Wire Wire Line
-	6250 1850 5750 1850
-Wire Wire Line
-	5750 1850 5750 1350
-Wire Wire Line
-	5750 1350 3400 1350
-Wire Wire Line
-	3400 1350 3400 1950
-Wire Wire Line
-	3400 2550 3400 2450
-Wire Wire Line
-	3400 3150 3400 2950
-Wire Wire Line
-	5900 1950 6250 1950
-Connection ~ 4000 1750
-Wire Wire Line
-	4000 1750 4000 2100
-Wire Wire Line
-	4000 2100 4100 2100
-Wire Wire Line
-	6750 3800 6750 3900
-Connection ~ 5450 1750
-Wire Wire Line
-	5450 2250 5900 2250
-Wire Wire Line
-	1400 3950 1400 3700
-Wire Wire Line
-	1400 3700 1250 3700
-Wire Wire Line
-	5450 3500 6350 3500
-Wire Wire Line
-	2150 1900 2150 1650
-Connection ~ 8000 3900
-Wire Wire Line
-	10150 2250 9250 2250
-Wire Wire Line
-	9250 2250 9250 3500
-Wire Wire Line
-	1250 3200 1900 3200
-Wire Wire Line
-	1900 3200 1900 1550
-Wire Wire Line
-	1900 1550 6250 1550
-Wire Wire Line
-	1250 3400 2150 3400
-Wire Wire Line
-	2150 1650 6250 1650
-Connection ~ 4750 2100
-Wire Wire Line
-	4600 2100 4750 2100
-Connection ~ 3600 3500
-Wire Wire Line
-	3600 3500 3600 1750
-Connection ~ 7400 3500
-Wire Wire Line
-	8000 3900 8000 3800
-Wire Wire Line
-	4950 1750 6250 1750
-Connection ~ 7400 3900
-Connection ~ 6150 3500
-Connection ~ 6750 3900
-Wire Wire Line
-	4750 2150 4750 2050
-Wire Wire Line
-	3600 1750 4550 1750
-Wire Wire Line
-	9250 3500 8400 3500
-Wire Wire Line
-	4450 3600 4450 3500
-Wire Wire Line
-	7150 3500 7600 3500
-Connection ~ 4450 3500
-Wire Wire Line
-	1250 3500 2800 3500
-Wire Wire Line
-	1250 3100 1750 3100
-Wire Wire Line
-	1750 3100 1750 1450
-Wire Wire Line
-	1750 1450 6250 1450
-Wire Wire Line
-	8950 2350 8950 2150
-Wire Wire Line
-	8950 2150 10150 2150
-Wire Wire Line
-	2150 3400 2150 2300
-Connection ~ 1750 3400
-Wire Wire Line
-	9000 3900 6150 3900
-Connection ~ 9000 3500
-Connection ~ 8600 3500
-Connection ~ 8600 3900
-Wire Wire Line
-	4450 4000 4450 4100
-Wire Wire Line
-	9000 3900 9000 4000
-Wire Wire Line
-	6150 3900 6150 4000
-Connection ~ 5450 2250
-Wire Wire Line
-	5450 2350 5450 2150
-Wire Wire Line
-	1250 3300 3800 3300
-Wire Wire Line
-	3900 3050 3800 3050
-Wire Wire Line
-	10150 2650 9850 2650
-Wire Wire Line
-	9850 2650 9850 4400
-Wire Wire Line
-	9850 4400 3500 4400
-Wire Wire Line
-	1250 3600 2350 3600
-Wire Wire Line
-	2350 3600 2350 3250
-Wire Wire Line
-	2350 2750 3100 2750
-Wire Wire Line
-	2700 3050 2550 3050
-Wire Wire Line
-	2550 3050 2550 2750
-Connection ~ 2550 2750
-Wire Wire Line
-	3800 3050 3800 3300
-Wire Wire Line
-	4750 3250 4750 3300
-Wire Wire Line
-	4750 2650 4750 2850
-Connection ~ 5250 1750
-Wire Wire Line
-	5350 2850 5250 2850
-Connection ~ 5250 2850
-Wire Wire Line
-	5250 3200 5250 1750
-Wire Wire Line
-	9300 3000 9250 3000
-Connection ~ 9250 3000
 $Comp
 L R R1
 U 1 1 508A6768
-P 9550 3000
-F 0 "R1" V 9630 3000 50  0000 C CNN
-F 1 "5K1" V 9550 3000 50  0000 C CNN
-	1    9550 3000
+P 3250 4400
+F 0 "R1" V 3330 4400 50  0000 C CNN
+F 1 "5K1" V 3250 4400 50  0000 C CNN
+	1    3250 4400
 	0    -1   -1   0
-$EndComp
-$Comp
-L DIODESCH D2
-U 1 1 508A66B2
-P 3300 4400
-F 0 "D2" H 3300 4500 40  0000 C CNN
-F 1 "DIODESCH" H 3300 4300 40  0000 C CNN
-	1    3300 4400
-	-1   0    0    -1
 $EndComp
 $Comp
@@
 	1    0    0    -1
 $EndComp
+Text Label 1350 3000 0    60   ~ 0
+Rx
 Text Label 1350 3100 0    60   ~ 0
-Rx
-Text Label 1350 3200 0    60   ~ 0
 Tx
 Text Notes 6250 2150 0    60   ~ 0
@@
 $EndComp
 $Comp
-L CONN_7 P1
+L CONN_8 P1
 U 1 1 504D1054
-P 900 3400
-F 0 "P1" V 850 3400 60  0000 C CNN
-F 1 "G9X" V 950 3400 60  0000 C CNN
-	1    900  3400
-	-1   0    0    1
-$EndComp
+P 900 3350
+F 0 "P1" V 850 3350 60  0000 C CNN
+F 1 "G9X" V 950 3350 60  0000 C CNN
+	1    900  3350
+	-1   0    0    1
+$EndComp
