File: hardware/pcb/gruvin9x.sch (KiCad schematic (older format))
At the start: 259 parts, among them IC1 ATMEGA2560-A_GRUVIN, J1 JUMPER_2W, J4 JUMPER_2W, K1 CONN_3, K2 CONN_3, K3 CONN_3, K4 CONN_5, K5 CONN_3, K6 CONN_3, P1 CONN_3X2, P10 CONN_5X2, P12 CONN_4, P13 CONN_8, P14 CONN_2, P15 CONN_4, P18 CONN_2, P2 CONN_5, P20 CONN_8, P21 CONN_3, P23 CONN_1, P24 CONN_1, P25 CONN_1, P26 CONN_1, P3 CONN_6, P4 CONN_9, P5 CONN_9, P6 CONN_6, P7 CONN_12, P8 CONN_30_LCD_GRUVIN, P9 CONN_1, Q1 BC847C, Q10 Si2319DS, Q2 BC847C, Q3 BC857C, Q4 BC847C, Q5 BC847C, Q6 Si2319DS, Q7 BC847C, Q8 BC847C, Q9 BC847C, SW1 SW_PUSH, SW2 SW_PUSH, SW3 SW_PUSH, SW4 SW_PUSH, SW5 SW_PUSH, SW6 SW_PUSH, U1 78L05, U2 78L05, U3 LN-6206-30, U4 TPS77601, U5 REF3012, X1 16MHz

Commit message: Apparently, my previous commit of the v4.2 frozen folder did not complete successfully, but I didn't realise. :/ This is a recommit of that -- but with changes as follows ...
. Added R118 in series with C63 to fix intermittent fault with soft-off
  circuitry. (Credit and thanks to x3mfly for this discovery and debug.)
. Added the AGND 'component' to the gruvin.lib shared module library. It 
  was missing for some reason, which was noticed when the net name for 
  AGND didn't seem to exist in PCBNEW, which in turn caused some brief
  confusion when re-laying tracks for R118.
. The above was all done in the so-called 'frozen' folder, s the changes
  were copied back to our current trunk/hardware/pcb folder.
. Miraculously (Cam) I remembered to update the gruvin9x-readme.txt file! :-D
Parts:
- added R118: 10K, symbol R
Connections:
- wire segments 725 -> 728

Commit message: Pad added to allow easier connection to C-of-Q9 for short-to-ground power-on at trainer jack, should it be required.
Production files including updated BOM (for R118) still to come.
Parts:
- added P11: CONN_1, symbol CONN_1

Commit message: ================================ = Differences V4.1a to V4.2b/c = ================================
PCB
===
-- Gruvin --
. Added tracks to links pins 1 & 2 on both J1 and J4. In the unlikely event
  anyone ever wants the opposite option for either jumper, they can break the 
  track. This will save time as well as the slightly unsightly solder-blob 
  bridges I've been doing on all the retail boards to date.
. v4.2c -- changed solder mask clearance to 0.0000, having been advised to
  let the factory use their own process-ideal clearances. This will mostly
  help for the 0.5mm pitch MCU and LCD socket parts.
Connections:
- wire segments 728 -> 729
Other:
- note added: "Default 1-2\nBreak track to change"
